File: SolenoidX13.sch (EAGLE design)
At the start: 0 parts

Commit message: owo
Parts:
- added C1, C10, C2, C7, C8, C9: 4.7uF, SparkFun-Capacitors:4.7UF0603
- added C11: 0.1uF, SparkFun-Capacitors:0.1UF-0603-25V-(+80/-20%)
- added C3, C4: 100nF, SparkFun-Capacitors:4.7UF0603
- added C5: 0.01uF, SparkFun-Capacitors:4.7UF0603
- added C6: 1uF, SparkFun-Capacitors:4.7UF0603
- added D1, D2, D4: (no value), SparkFun-LED:LED0603
- added J1, J3, J4: (no value), SparkFun-Connectors:CONN_02
- added R1, R2, R3: 1k, SparkFun-Resistors:1KOHM-0603-1/10W-1%
- added R10, R11: 60, SparkFun-Resistors:1KOHM-0603-1/10W-1%
- added R4, R6, R7: (no value), SparkFun-Resistors:RESISTOR0603
- added RESET: SWITCH, DiscreteComponents:SWITCH
- added SV1: (no value), con-lsta:FE05-1
- added U$3: STM32F042K6T6, PI_Shield_Library:STM32F042K6T6
- added U$8: TCAN337D, PI_Shield_Library:TCAN337D
- added U1: ULN2003V12, ULN2003V12:ULN2003V12
- added Y1: ECS-80-S-4X, ECS-80-S-4X:ECS-80-S-4X
Connections:
- new net +3V3: C1.1, C10.1, C2.1, C3.1, C4.1, C5.1, C6.1, R2.2, R6.2, SV1.5, U$3.VDD, U$3.VDDA, U$3.VDDIO2, U$8.VCC
- new net 12V: J3.2, R4.2, U1.COM
- new net 3.3V: J1.2
- new net CAN_H: J4.2, R10.2, U$8.CANH
- new net CAN_L: J4.1, R11.1, U$8.CANL
- new net CAN_RX: U$3.PA11, U$8.RXD
- new net CAN_TX: U$3.PA12, U$8.TXD
- new net GND: C1.2, C10.2, C11.1, C2.2, C3.2, C4.2, C5.2, C6.2, C7.2, C8.2, C9.2, D1.C, D2.C, D4.C, J1.1, J3.1, RESET.P$1, SV1.3, U$3.PB8-BOOT0, U$3.VSS, U$3.VSS1, U$8.GND, U1.GND
- new net GPIO0: U$3.PB7
- new net GPIO1: U$3.PB6, U1.IN4
- new net GPIO10: U$3.PA5, U1.IN3
- new net GPIO11: U$3.PA6, U1.IN2
- new net GPIO12: U$3.PA7, U1.IN1
- new net GPIO13: U$3.PA8
- new net GPIO14: U$3.PA9
- new net GPIO15: U$3.PA10
- new net GPIO2: U$3.PB4, U1.IN5
- new net GPIO3: U$3.PB3, U1.IN6
- new net GPIO8: U$3.PA3
- new net GPIO9: U$3.PA4
- new net LED: R7.2, U$3.PA15
- new net N$1: C9.1, R1.1, Y1.2
- new net N$2: C8.1, R3.1, Y1.1
- new net N$24: D1.A, R7.1
- new net N$25: D4.A, R4.1
- new net N$27: D2.A, R6.1
- new net N$5: C11.2, R10.1, R11.2
- new net NRST: SV1.1
- new net NRST1: C7.1, R2.1, RESET.P$2, U$3.NRST
- new net OSC_IN: R3.2, U$3.PF0-OSC_IN
- new net OSC_OUT: R1.2, U$3.PF1-OSC_OUT
- new net SOL1_1: U1.OUT1
- new net SOL2_1: U1.OUT2
- new net SOL3_1: U1.OUT3
- new net SOL4_1: U1.OUT4
- new net SOL5_1: U1.OUT5
- new net SOL6_1: U1.OUT6
- new net SWCLK: SV1.4, U$3.PA14
- new net SWDIO: SV1.2, U$3.PA13
Other:
- note added: "CAN"
- note added: "CAN TERMINATION"
- note added: "CAN TRANSCEIVER"
- note added: "NPN Array"
- note added: "Pin 1 (VDD)"
- note added: "Pin 17 (VDDIO2)"
- note added: "Pin 5 (VDDA)"
- note added: "Power Indication LEDs"
- note added: "STM"
- note added: "Solenoid Output Connector"
- note added: "T21 Connector for 12V, CAN, GND, 3.3V"

Commit message: owo?
Parts:
- removed C8, C9: 4.7uF, SparkFun-Capacitors:4.7UF0603
- removed R4, R6: (no value), SparkFun-Resistors:RESISTOR0603
- removed Y1: ECS-80-S-4X, ECS-80-S-4X:ECS-80-S-4X
- R1: value 1k -> 680; device SparkFun-Resistors:1KOHM-0603-1/10W-1% -> SparkFun-Resistors:680OHM-0603-1/10W-5%
- R10, R11: value 60 -> 1k
- R3: value 1k -> 82; device SparkFun-Resistors:1KOHM-0603-1/10W-1% -> SparkFun-Resistors:82OHM-0603-1/10W-1%
Connections:
- removed net GPIO2: U$3.PB4, U1.IN5
- removed net GPIO3: U$3.PB3, U1.IN6
- removed net N$1: C9.1, R1.1, Y1.2
- removed net N$2: C8.1, R3.1, Y1.1
- removed net OSC_IN: R3.2, U$3.PF0-OSC_IN
- removed net OSC_OUT: R1.2, U$3.PF1-OSC_OUT
- new net GPIO4: U1.IN4
- new net GPIO5: U$3.PA2, U1.IN2, U1.IN5
- new net GPIO6: U$3.PA3, U1.IN3, U1.IN6
- net +3V3: now also R3.2; no longer R6.2
- net 12V: now also R1.2; no longer R4.2
- net GND: no longer C8.2, C9.2
- net GPIO0: now also U$3.PA1; no longer U$3.PB7
- net GPIO1: now also U$3.PA0, U1.IN1; no longer U$3.PB6, U1.IN4
- net GPIO10: now also U$3.PA7; no longer U$3.PA5, U1.IN3
- net GPIO11: now also U$3.PB0; no longer U$3.PA6, U1.IN2
- net GPIO12: now also U$3.PB1; no longer U$3.PA7, U1.IN1
- net GPIO8: now also U$3.PA5; no longer U$3.PA3
- net GPIO9: now also U$3.PA6; no longer U$3.PA4
- net N$25: now also R1.1; no longer R4.1
- net N$27: now also R3.1; no longer R6.1

Commit message: hi
Connections:
- removed net GPIO10: U$3.PA7
- removed net GPIO11: U$3.PB0
- removed net GPIO12: U$3.PB1
- removed net GPIO13: U$3.PA8
- removed net GPIO14: U$3.PA9
- removed net GPIO15: U$3.PA10
- removed net GPIO8: U$3.PA5
- removed net GPIO9: U$3.PA6
- new net GPIO2: U$3.PA2, U1.IN2
- new net GPIO3: U$3.PA3, U1.IN3
- net GPIO0: now also U$3.PA0; no longer U$3.PA1
- net GPIO1: now also U$3.PA1; no longer U$3.PA0
- net GPIO4: now also U$3.PA4
- net GPIO5: now also U$3.PA5; no longer U$3.PA2, U1.IN2
- net GPIO6: now also U$3.PA6; no longer U$3.PA3, U1.IN3
Changed lines of the file:
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@@
-</segment>
-</net>
-<net name="GPIO15" class="0">
-<segment>
-<pinref part="U$3" gate="G$1" pin="PA10"/>
-<wire x1="132.08" y1="104.14" x2="147.32" y2="104.14" width="0.1524" layer="91"/>
-<label x="144.78" y="104.14" size="1.778" layer="95"/>
-</segment>
-</net>
-<net name="GPIO14" class="0">
-<segment>
-<pinref part="U$3" gate="G$1" pin="PA9"/>
-<wire x1="132.08" y1="101.6" x2="147.32" y2="101.6" width="0.1524" layer="91"/>
-<label x="144.78" y="101.6" size="1.778" layer="95"/>
-</segment>
-</net>
-<net name="GPIO13" class="0">
-<segment>
-<pinref part="U$3" gate="G$1" pin="PA8"/>
-<wire x1="132.08" y1="99.06" x2="147.32" y2="99.06" width="0.1524" layer="91"/>
-<label x="144.78" y="99.06" size="1.778" layer="95"/>
 </segment>
 </net>
 <net name="GPIO1" class="0">
+<segment>
+<wire x1="86.36" y1="99.06" x2="81.28" y2="99.06" width="0.1524" layer="91"/>
+<label x="83.82" y="99.06" size="1.778" layer="95" rot="R180"/>
+<pinref part="U$3" gate="G$1" pin="PA1"/>
+</segment>
+</net>
+<net name="GPIO0" class="0">
 <segment>
 <wire x1="86.36" y1="101.6" x2="81.28" y2="101.6" width="0.1524" layer="91"/>
@@
 </segment>
 </net>
-<net name="GPIO0" class="0">
-<segment>
-<wire x1="86.36" y1="99.06" x2="81.28" y2="99.06" width="0.1524" layer="91"/>
-<label x="83.82" y="99.06" size="1.778" layer="95" rot="R180"/>
-<pinref part="U$3" gate="G$1" pin="PA1"/>
-</segment>
-</net>
-<net name="GPIO5" class="0">
+<net name="GPIO6" class="0">
+<segment>
+<wire x1="106.68" y1="73.66" x2="106.68" y2="83.82" width="0.1524" layer="91"/>
+<label x="106.68" y="73.66" size="1.778" layer="95" rot="R90"/>
+<pinref part="U$3" gate="G$1" pin="PA6"/>
+</segment>
+</net>
+<net name="GPIO2" class="0">
 <segment>
 <wire x1="86.36" y1="96.52" x2="81.28" y2="96.52" width="0.1524" layer="91"/>
@@
 </segment>
 </net>
-<net name="GPIO12" class="0">
-<segment>
-<wire x1="116.84" y1="83.82" x2="116.84" y2="73.66" width="0.1524" layer="91"/>
-<label x="116.84" y="73.66" size="1.778" layer="95" rot="R90"/>
-<pinref part="U$3" gate="G$1" pin="PB1"/>
-</segment>
-</net>
-<net name="GPIO10" class="0">
-<segment>
-<wire x1="111.76" y1="83.82" x2="111.76" y2="73.66" width="0.1524" layer="91"/>
-<label x="111.76" y="73.66" size="1.778" layer="95" rot="R90"/>
-<pinref part="U$3" gate="G$1" pin="PA7"/>
-</segment>
-</net>
-<net name="GPIO11" class="0">
-<segment>
-<wire x1="114.3" y1="83.82" x2="114.3" y2="73.66" width="0.1524" layer="91"/>
-<label x="114.3" y="73.66" size="1.778" layer="95" rot="R90"/>
-<pinref part="U$3" gate="G$1" pin="PB0"/>
-</segment>
-</net>
-<net name="GPIO9" class="0">
-<segment>
-<wire x1="106.68" y1="83.82" x2="106.68" y2="73.66" width="0.1524" layer="91"/>
-<label x="106.68" y="73.66" size="1.778" layer="95" rot="R90"/>
-<pinref part="U$3" gate="G$1" pin="PA6"/>
-</segment>
-</net>
-<net name="GPIO8" class="0">
-<segment>
-<wire x1="104.14" y1="83.82" x2="104.14" y2="73.66" width="0.1524" layer="91"/>
-<label x="104.14" y="73.66" size="1.778" layer="95" rot="R90"/>
-<pinref part="U$3" gate="G$1" pin="PA5"/>
-</segment>
-</net>
-<net name="GPIO6" class="0">
+<net name="GPIO3" class="0">
 <segment>
 <wire x1="99.06" y1="73.66" x2="99.06" y2="83.82" width="0.1524" layer="91"/>
 <label x="99.06" y="73.66" size="1.778" layer="95" rot="R90"/>
 <pinref part="U$3" gate="G$1" pin="PA3"/>
+</segment>
+</net>
+<net name="GPIO4" class="0">
+<segment>
+<wire x1="101.6" y1="73.66" x2="101.6" y2="83.82" width="0.1524" layer="91"/>
+<label x="101.6" y="73.66" size="1.778" layer="95" rot="R90"/>
+<pinref part="U$3" gate="G$1" pin="PA4"/>
+</segment>
+</net>
+<net name="GPIO5" class="0">
+<segment>
+<wire x1="104.14" y1="73.66" x2="104.14" y2="83.82" width="0.1524" layer="91"/>
+<label x="104.14" y="73.66" size="1.778" layer="95" rot="R90"/>
+<pinref part="U$3" gate="G$1" pin="PA5"/>
 </segment>
 </net>
@@
 <net name="GPIO6" class="0">
 <segment>
+<wire x1="40.64" y1="78.74" x2="33.02" y2="78.74" width="0.1524" layer="91"/>
+<label x="33.02" y="78.74" size="1.778" layer="95"/>
+<pinref part="U1" gate="G$1" pin="IN6"/>
+</segment>
+</net>
+<net name="GPIO5" class="0">
+<segment>
+<wire x1="40.64" y1="83.82" x2="33.02" y2="83.82" width="0.1524" layer="91"/>
+<label x="33.02" y="83.82" size="1.778" layer="95"/>
+<pinref part="U1" gate="G$1" pin="IN5"/>
+</segment>
+</net>
+<net name="GPIO4" class="0">
+<segment>
+<wire x1="40.64" y1="88.9" x2="33.02" y2="88.9" width="0.1524" layer="91"/>
+<label x="33.02" y="88.9" size="1.778" layer="95"/>
+<pinref part="U1" gate="G$1" pin="IN4"/>
+</segment>
+</net>
+<net name="GPIO3" class="0">
+<segment>
 <wire x1="40.64" y1="93.98" x2="33.02" y2="93.98" width="0.1524" layer="91"/>
 <label x="33.02" y="93.98" size="1.778" layer="95"/>
 <pinref part="U1" gate="G$1" pin="IN3"/>
 </segment>
-<segment>
-<wire x1="40.64" y1="78.74" x2="33.02" y2="78.74" width="0.1524" layer="91"/>
-<label x="33.02" y="78.74" size="1.778" layer="95"/>
-<pinref part="U1" gate="G$1" pin="IN6"/>
-</segment>
-</net>
-<net name="GPIO5" class="0">
+</net>
+<net name="GPIO2" class="0">
 <segment>
 <wire x1="40.64" y1="99.06" x2="33.02" y2="99.06" width="0.1524" layer="91"/>
@@
 <pinref part="U1" gate="G$1" pin="IN2"/>
 </segment>
-<segment>
-<wire x1="40.64" y1="83.82" x2="33.02" y2="83.82" width="0.1524" layer="91"/>
-<label x="33.02" y="83.82" size="1.778" layer="95"/>
-<pinref part="U1" gate="G$1" pin="IN5"/>
-</segment>
-</net>
-<net name="GPIO4" class="0">
-<segment>
-<wire x1="40.64" y1="88.9" x2="33.02" y2="88.9" width="0.1524" layer="91"/>
-<label x="33.02" y="88.9" size="1.778" layer="95"/>
-<pinref part="U1" gate="G$1" pin="IN4"/>
-</segment>
-</net>
+</net>

Commit message: board is done lol
Parts:
- removed J3, J4: (no value), SparkFun-Connectors:CONN_02
- J1: value (none) -> SAMTEC-CLT-111-01-X-DJ; device SparkFun-Connectors:CONN_02 -> SAMTEC-CLT-111-01-X-D:SAMTEC-CLT-111-01-X-DJ
Connections:
- removed net 3.3V: J1.2
- new net ALERT1: J1.18, U$3.PB4
- new net ALERT2: J1.17, U$3.PB3
- new net C2_1: J1.16, U$3.PB0
- new net C2_2: J1.15, U$3.PB1
- new net CLK: J1.20, U$3.PA9
- new net DATA: J1.22, U$3.PA10
- new net GPIO7: U$3.PA7
- net +3V3: now also J1.6
- net 12V: now also J1.11; no longer J3.2
- net CAN_H: now also J1.19; no longer J4.2
- net CAN_L: now also J1.21; no longer J4.1
- net GND: now also J1.10, J1.12, J1.4, J1.8; no longer J1.1, J3.1
- net SOL1_1: now also J1.2
- net SOL2_1: now also J1.1
- net SOL3_1: now also J1.3
- net SOL4_1: now also J1.5
- net SOL5_1: now also J1.7
- net SOL6_1: now also J1.9
- net SWCLK: now also U$3.PA13; no longer U$3.PA14
- net SWDIO: now also U$3.PA14; no longer U$3.PA13
Other:
- note added: "Connectors Owo"
- note removed: "Solenoid Output Connector"
- note removed: "T21 Connector for 12V, CAN, GND, 3.3V"

Commit message: lol
Parts:
- removed RESET: SWITCH, DiscreteComponents:SWITCH
- added U$1: (no value), Push button - FSM2JMTR:DISCRETECOMPONENTS_SWITCH
Connections:
- net GND: now also U$1.P$1; no longer RESET.P$1
- net NRST1: now also U$1.P$2; no longer RESET.P$2
Changed lines of the file:
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@@
 <layer number="115" name="ReferenceISLANDS" color="7" fill="1" visible="no" active="yes"/>
 <layer number="116" name="Patch_BOT" color="9" fill="4" visible="yes" active="yes"/>
+<layer number="117" name="mPads" color="7" fill="1" visible="yes" active="yes"/>
 <layer number="118" name="Rect_Pads" color="7" fill="1" visible="no" active="yes"/>
+<layer number="119" name="mUnrouted" color="7" fill="1" visible="yes" active="yes"/>
+<layer number="120" name="mDimension" color="7" fill="1" visible="yes" active="yes"/>
 <layer number="121" name="_tsilk" color="7" fill="1" visible="yes" active="yes"/>
 <layer number="122" name="_bsilk" color="7" fill="1" visible="yes" active="yes"/>
@@
 <layer number="128" name="_bValues" color="7" fill="1" visible="yes" active="yes"/>
 <layer number="129" name="Mask" color="7" fill="1" visible="yes" active="yes"/>
+<layer number="130" name="mbStop" color="7" fill="1" visible="yes" active="yes"/>
 <layer number="131" name="tAdjust" color="7" fill="1" visible="yes" active="yes"/>
 <layer number="132" name="bAdjust" color="7" fill="1" visible="yes" active="yes"/>
+<layer number="133" name="mtFinish" color="7" fill="1" visible="yes" active="yes"/>
+<layer number="134" name="mbFinish" color="7" fill="1" visible="yes" active="yes"/>
+<layer number="135" name="mtGlue" color="7" fill="1" visible="yes" active="yes"/>
+<layer number="136" name="mbGlue" color="7" fill="1" visible="yes" active="yes"/>
+<layer number="137" name="mtTest" color="7" fill="1" visible="yes" active="yes"/>
+<layer number="138" name="mbTest" color="7" fill="1" visible="yes" active="yes"/>
+<layer number="139" name="mtKeepout" color="7" fill="1" visible="yes" active="yes"/>
+<layer number="140" name="mbKeepout" color="7" fill="1" visible="yes" active="yes"/>
+<layer number="141" name="mtRestrict" color="7" fill="1" visible="yes" active="yes"/>
+<layer number="142" name="mbRestrict" color="7" fill="1" visible="yes" active="yes"/>
+<layer number="143" name="mvRestrict" color="7" fill="1" visible="yes" active="yes"/>
 <layer number="144" name="Drill_legend" color="7" fill="1" visible="yes" active="yes"/>
+<layer number="145" name="mHoles" color="7" fill="1" visible="yes" active="yes"/>
+<layer number="146" name="mMilling" color="7" fill="1" visible="yes" active="yes"/>
+<layer number="147" name="mMeasures" color="7" fill="1" visible="yes" active="yes"/>
+<layer number="148" name="mDocument" color="7" fill="1" visible="yes" active="yes"/>
+<layer number="149" name="mReference" color="7" fill="1" visible="yes" active="yes"/>
 <layer number="150" name="Notes" color="7" fill="1" visible="yes" active="yes"/>
 <layer number="151" name="HeatSink" color="7" fill="1" visible="yes" active="yes"/>
@@
 <layer number="154" name="FabDoc2" color="7" fill="1" visible="yes" active="yes"/>
 <layer number="155" name="FabDoc3" color="7" fill="1" visible="yes" active="yes"/>
+<layer number="191" name="mNets" color="7" fill="1" visible="yes" active="yes"/>
+<layer number="192" name="mBusses" color="7" fill="1" visible="yes" active="yes"/>
+<layer number="193" name="mPins" color="7" fill="1" visible="yes" active="yes"/>
+<layer number="194" name="mSymbols" color="7" fill="1" visible="yes" active="yes"/>
+<layer number="195" name="mNames" color="7" fill="1" visible="yes" active="yes"/>
+<layer number="196" name="mValues" color="7" fill="1" visible="yes" active="yes"/>
 <layer number="199" name="Contour" color="7" fill="1" visible="yes" active="yes"/>
 <layer number="200" name="200bmp" color="1" fill="10" visible="yes" active="yes"/>
@@
 <part name="C7" library="SparkFun-Capacitors" library_urn="urn:adsk.eagle:library:510" deviceset="4.7UF" device="0603" package3d_urn="urn:adsk.eagle:package:37414/1" value="4.7uF"/>
 <part name="GND3" library="supply2" library_urn="urn:adsk.eagle:library:372" deviceset="GND" device=""/>
-<part name="RESET" library="DiscreteComponents" deviceset="SWITCH" device="" value=""/>
 <part name="R2" library="SparkFun-Resistors" library_urn="urn:adsk.eagle:library:532" deviceset="1KOHM" device="-0603-1/10W-1%" package3d_urn="urn:adsk.eagle:package:39650/1" value="1k"/>
 <part name="+3V2" library="supply1" library_urn="urn:adsk.eagle:library:371" deviceset="+3V3" device=""/>
@@
 <part name="J1" library="SAMTEC-CLT-111-01-X-D" deviceset="SAMTEC-CLT-111-01-X-D" device="J"/>
 <part name="SV1" library="con-lsta" library_urn="urn:adsk.eagle:library:161" deviceset="FE05-1" device="" package3d_urn="urn:adsk.eagle:package:8190/1"/>
+<part name="U$1" library="Push button - FSM2JMTR" deviceset="DISCRETECOMPONENTS_SWITCH" device="" package3d_urn="urn:adsk.eagle:package:24384574/2"/>
 </parts>
 <sheets>
@@
 <attribute name="VALUE" x="31.115" y="85.725" size="1.778" layer="96"/>
 </instance>
-<instance part="RESET" gate="G$1" x="45.72" y="101.6" smashed="yes" rot="R90"/>
 <instance part="R2" gate="G$1" x="33.02" y="119.38" smashed="yes" rot="R90">
 <attribute name="NAME" x="31.496" y="119.38" size="1.778" layer="95" font="vector" rot="R90" align="bottom-center"/>
@@
 <attribute name="VALUE" x="68.58" y="116.84" size="1.778" layer="96" rot="R90"/>
 </instance>
+<instance part="U$1" gate="G$1" x="45.72" y="101.6" smashed="yes" rot="R90"/>
 </instances>
 <busses>
@@
 <pinref part="C7" gate="G$1" pin="2"/>
 <wire x1="33.02" y1="91.44" x2="33.02" y2="93.98" width="0.1524" layer="91"/>
-<pinref part="RESET" gate="G$1" pin="P$1"/>
 <wire x1="33.02" y1="93.98" x2="33.02" y2="96.52" width="0.1524" layer="91"/>
 <wire x1="45.72" y1="93.98" x2="33.02" y2="93.98" width="0.1524" layer="91"/>
 <junction x="33.02" y="93.98"/>
+<pinref part="U$1" gate="G$1" pin="P$1"/>
 </segment>
 <segment>
@@
 <pinref part="C7" gate="G$1" pin="1"/>
 <pinref part="R2" gate="G$1" pin="1"/>
-<pinref part="RESET" gate="G$1" pin="P$2"/>
 <wire x1="33.02" y1="109.22" x2="33.02" y2="104.14" width="0.1524" layer="91"/>
 <junction x="33.02" y="109.22"/>
 <pinref part="U$3" gate="G$1" pin="NRST"/>
+<wire x1="33.02" y1="109.22" x2="45.72" y2="109.22" width="0.1524" layer="91"/>
 <wire x1="45.72" y1="109.22" x2="86.36" y2="109.22" width="0.1524" layer="91"/>
+<wire x1="33.02" y1="114.3" x2="33.02" y2="109.22" width="0.1524" layer="91"/>
+<pinref part="U$1" gate="G$1" pin="P$2"/>
 <junction x="45.72" y="109.22"/>
-<wire x1="33.02" y1="114.3" x2="33.02" y2="109.22" width="0.1524" layer="91"/>
-<wire x1="45.72" y1="109.22" x2="33.02" y2="109.22" width="0.1524" layer="91"/>
-</segment>
-</net>
+</segment>
+</net>
