File: SolenoidX13.sch (EAGLE design)
At the start: 23 parts, among them U1 ULN2003V12

Commit message: big pog uwu
Connections:
- net SWCLK: now also STM.PA14; no longer STM.PA13
- net SWDIO: now also STM.PA13; no longer STM.PA14
Changed lines of the file:
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@@
 </segment>
 </net>
-<net name="SWDIO" class="0">
+<net name="SWCLK" class="0">
 <segment>
 <wire x1="116.84" y1="104.14" x2="132.08" y2="104.14" width="0.1524" layer="91"/>
@@
 </segment>
 </net>
-<net name="SWCLK" class="0">
+<net name="SWDIO" class="0">
 <segment>
 <wire x1="116.84" y1="101.6" x2="132.08" y2="101.6" width="0.1524" layer="91"/>

Commit message: New SWD programming connecotr
Parts:
- removed C4, C6: 4.7uF, SparkFun-Capacitors:4.7UF0603
- C10, C2, C3, C5, C7: value 4.7uF -> 0.1uF
- R2: value 1k -> 10k
- SV1: value (none) -> 3V3 -SWCLK-GND-SWDIO- NRST; device con-lsta:FE05-1 -> CONN, Serial Wire Programming Headers:SWD_CONN
Connections:
- net +3V3: now also SV1.3V3; no longer C4.1, C6.1, SV1.5
- net GND: now also SV1.GND; no longer C4.2, C6.2, SV1.3
- net NRST: now also SV1.NRST; no longer SV1.1
- net SWCLK: now also SV1.SWCLK; no longer SV1.4
- net SWDIO: now also SV1.SWDIO; no longer SV1.2
