File: SolenoidX13.brd (EAGLE design)
At the start: 24.3 x 25.4 mm, 26 parts, among them J1 SAMTEC-CLT-111-01-X-DJ, U1 ULN2003V12

Commit message: final
Parts:
- moved R5 2.35 mm to (6.76, 10.9), turned to 270 degrees
- moved R4 0.80 mm to (8.64, 7.70)
Routing:
- net N$1: track 6.49 -> 7.81 mm
- net N$2: track 5.91 -> 7.17 mm
- net C2_1: track 6.81 -> 5.59 mm
Changed lines of the file:
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@@
 <attribute name="VALUE" x="24.0792" y="17.0942" size="1.27" layer="27" rot="R90" align="top-center"/>
 </element>
-<element name="R4" library="SparkFun-Resistors" library_urn="urn:adsk.eagle:library:532" package="0603" package3d_urn="urn:adsk.eagle:package:39650/1" value="4.7k" x="8.89" y="8.4582" smashed="yes" rot="R180">
-<attribute name="NAME" x="8.89" y="7.6962" size="0.6096" layer="25" font="vector" ratio="20" rot="R180" align="bottom-center"/>
-<attribute name="PROD_ID" value="RES-07857" x="8.89" y="8.4582" size="1.778" layer="27" rot="R180" display="off"/>
-<attribute name="VALUE" x="8.89" y="9.2202" size="0.6096" layer="27" font="vector" ratio="20" rot="R180" align="top-center"/>
+<element name="R4" library="SparkFun-Resistors" library_urn="urn:adsk.eagle:library:532" package="0603" package3d_urn="urn:adsk.eagle:package:39650/1" value="4.7k" x="8.636" y="7.6962" smashed="yes" rot="R180">
+<attribute name="NAME" x="8.636" y="6.9342" size="0.6096" layer="25" font="vector" ratio="20" rot="R180" align="bottom-center"/>
+<attribute name="PROD_ID" value="RES-07857" x="8.636" y="7.6962" size="1.778" layer="27" rot="R180" display="off"/>
+<attribute name="VALUE" x="8.636" y="8.4582" size="0.6096" layer="27" font="vector" ratio="20" rot="R180" align="top-center"/>
 </element>
-<element name="R5" library="SparkFun-Resistors" library_urn="urn:adsk.eagle:library:532" package="0603" package3d_urn="urn:adsk.eagle:package:39650/1" value="4.7k" x="8.89" y="9.9568" smashed="yes" rot="R180">
-<attribute name="NAME" x="8.89" y="9.1948" size="0.6096" layer="25" font="vector" ratio="20" rot="R180" align="bottom-center"/>
-<attribute name="PROD_ID" value="RES-07857" x="8.636" y="9.9568" size="1.778" layer="27" rot="R180" display="off"/>
-<attribute name="VALUE" x="8.89" y="10.7188" size="0.6096" layer="27" font="vector" ratio="20" rot="R180" align="top-center"/>
+<element name="R5" library="SparkFun-Resistors" library_urn="urn:adsk.eagle:library:532" package="0603" package3d_urn="urn:adsk.eagle:package:39650/1" value="4.7k" x="6.7564" y="10.9474" smashed="yes" rot="R270">
+<attribute name="NAME" x="7.5184" y="10.9474" size="0.6096" layer="25" font="vector" ratio="20" rot="R270" align="bottom-center"/>
+<attribute name="PROD_ID" value="RES-07857" x="6.7564" y="10.6934" size="1.778" layer="27" rot="R270" display="off"/>
+<attribute name="VALUE" x="5.9944" y="10.9474" size="0.6096" layer="27" font="vector" ratio="20" rot="R270" align="top-center"/>
 </element>
 </elements>
@@
 <via x="11.509" y="22.733" extent="1-16" drill="0.35"/>
 <via x="12.779" y="24.0284" extent="1-16" drill="0.35"/>
-<via x="7.9784" y="12.0904" extent="1-16" drill="0.35"/>
+<via x="7.9784" y="11.0744" extent="1-16" drill="0.35"/>
 <wire x1="18.796" y1="16.5744" x2="18.7316" y2="16.51" width="0.508" layer="16"/>
 <wire x1="18.7316" y1="16.51" x2="17.2584" y2="16.51" width="0.508" layer="16"/>
@@
 <via x="13.2362" y="7.2136" extent="1-16" drill="0.35"/>
 <via x="13.4902" y="10.0076" extent="1-16" drill="0.35"/>
-<via x="9.9342" y="7.3152" extent="1-16" drill="0.35"/>
+<via x="8.6642" y="6.2992" extent="1-16" drill="0.35"/>
 </signal>
 <signal name="+3V3">
@@
 <wire x1="20.4401375" y1="20.3736" x2="20.1071375" y2="20.0406" width="0.4064" layer="1"/>
 <wire x1="20.1071375" y1="20.0406" x2="18.6302" y2="20.0406" width="0.4064" layer="1"/>
-<wire x1="18.6302" y1="20.0406" x2="18.6556" y2="20.0406" width="0.4064" layer="1"/>
-<wire x1="19.3967875" y1="19.422" x2="19.2742" y2="19.422" width="0.4064" layer="1"/>
-<wire x1="19.2742" y1="19.422" x2="18.6556" y2="20.0406" width="0.4064" layer="1"/>
+<wire x1="18.6302" y1="20.0406" x2="19.3967875" y2="20.0406" width="0.4064" layer="1"/>
+<wire x1="19.3967875" y1="19.422" x2="19.3967875" y2="20.0406" width="0.4064" layer="1"/>
 <via x="19.3967875" y="19.422" extent="1-16" drill="0.35"/>
 <wire x1="12.4088" y1="3.0380625" x2="12.6274625" y2="2.8194" width="0.4064" layer="16"/>
@@
 <signal name="C2_1">
 <contactref element="J1" pad="16"/>
-<wire x1="1.8418" y1="8.4714" x2="2.7938" y2="9.4234" width="0.254" layer="1"/>
+<wire x1="2.7938" y1="9.4234" x2="1.8418" y2="8.4714" width="0.254" layer="1"/>
 <contactref element="R5" pad="2"/>
-<wire x1="7.5066" y1="9.4234" x2="8.04" y2="9.9568" width="0.254" layer="1"/>
-<wire x1="2.7938" y1="9.4234" x2="7.5066" y2="9.4234" width="0.254" layer="1"/>
+<wire x1="6.7564" y1="10.0974" x2="6.0824" y2="9.4234" width="0.254" layer="1"/>
+<wire x1="6.0824" y1="9.4234" x2="2.7938" y2="9.4234" width="0.254" layer="1"/>
 </signal>
 <signal name="C2_2">
 <contactref element="J1" pad="15"/>
 <contactref element="R4" pad="2"/>
-<wire x1="8.04" y1="8.4582" x2="4.877" y2="8.4582" width="0.254" layer="1"/>
-<wire x1="4.877" y1="8.4582" x2="4.8638" y2="8.4714" width="0.254" layer="1"/>
+<wire x1="7.786" y1="7.6962" x2="6.782" y2="7.6962" width="0.254" layer="1"/>
+<wire x1="6.782" y1="7.6962" x2="6.0068" y2="8.4714" width="0.254" layer="1"/>
+<wire x1="6.0068" y1="8.4714" x2="4.8638" y2="8.4714" width="0.254" layer="1"/>
 </signal>
 <signal name="GPIO0">
@@
 <wire x1="11.5802" y1="13.7906" x2="11.063225" y2="13.7906" width="0.254" layer="1"/>
 <wire x1="11.063225" y1="13.7906" x2="10.65" y2="13.377375" width="0.254" layer="1"/>
-<wire x1="9.906" y1="8.4582" x2="9.74" y2="8.4582" width="0.254" layer="1"/>
-<wire x1="10.65" y1="13.377375" x2="10.65" y2="9.2022" width="0.254" layer="1"/>
-<wire x1="10.65" y1="9.2022" x2="9.906" y2="8.4582" width="0.254" layer="1"/>
+<wire x1="10.65" y1="13.377375" x2="10.65" y2="7.9322" width="0.254" layer="1"/>
+<wire x1="9.486" y1="7.6962" x2="10.414" y2="7.6962" width="0.254" layer="1"/>
+<wire x1="10.65" y1="7.9322" x2="10.414" y2="7.6962" width="0.254" layer="1"/>
 </signal>
 <signal name="N$2">
@@
 <contactref element="R5" pad="1"/>
 <wire x1="11.5802" y1="14.5906" x2="10.7044" y2="14.5906" width="0.254" layer="1"/>
-<wire x1="10.1854" y1="10.4022" x2="9.74" y2="9.9568" width="0.254" layer="1"/>
-<wire x1="10.7044" y1="14.5906" x2="10.1854" y2="14.0716" width="0.254" layer="1"/>
-<wire x1="10.1854" y1="14.0716" x2="10.1854" y2="10.4022" width="0.254" layer="1"/>
+<wire x1="10.1854" y1="14.0716" x2="10.7044" y2="14.5906" width="0.254" layer="1"/>
+<wire x1="8.802" y1="11.772" x2="6.7818" y2="11.772" width="0.254" layer="1"/>
+<wire x1="6.7564" y1="11.7974" x2="6.7818" y2="11.772" width="0.254" layer="1"/>
+<wire x1="8.802" y1="11.772" x2="8.9154" y2="11.6586" width="0.254" layer="1"/>
+<wire x1="8.9154" y1="11.6586" x2="9.6012" y2="11.6586" width="0.254" layer="1"/>
+<wire x1="9.6012" y1="11.6586" x2="10.1854" y2="12.2428" width="0.254" layer="1"/>
+<wire x1="10.1854" y1="12.2428" x2="10.1854" y2="14.0716" width="0.254" layer="1"/>
 </signal>
 </signals>

Commit message: pog
Routing:
- net CLK: track 16.8 -> 22.3 mm
- net GND: vias 23 -> 28
- added copper zone on layer 16, net NO
Changed lines of the file:
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@@
 <attribute name="NAME" x="11.4046" y="10.9728" size="0.6096" layer="26" font="vector" ratio="20" rot="MR0" align="bottom-center"/>
 <attribute name="PROD_ID" value="CAP-08280" x="14.7066" y="11.9888" size="1.778" layer="28" rot="MR0" display="off"/>
-<attribute name="VALUE" x="11.4046" y="9.4488" size="0.6096" layer="28" font="vector" ratio="20" rot="MR0" align="top-center"/>
+<attribute name="VALUE" x="11.4046" y="9.525" size="0.6096" layer="28" font="vector" ratio="20" rot="MR0" align="top-center"/>
 </element>
 <element name="C3" library="SparkFun-Capacitors" library_urn="urn:adsk.eagle:library:510" package="0603" package3d_urn="urn:adsk.eagle:package:37414/1" value="100nF" x="20.2946" y="17.4244" smashed="yes" rot="MR270">
@@
 <via x="19.6878" y="10.414" extent="1-16" drill="0.35"/>
 <via x="15.8016" y="4.6736" extent="1-16" drill="0.35"/>
-<via x="11.5344" y="6.7818" extent="1-16" drill="0.35"/>
+<via x="11.5344" y="6.604" extent="1-16" drill="0.35"/>
 <via x="17.0208" y="9.3218" extent="1-16" drill="0.35"/>
 <via x="6.6322" y="6.5786" extent="1-16" drill="0.35"/>
@@
 <via x="15.2936" y="13.462" extent="1-16" drill="0.35"/>
 <via x="17.9352" y="15.1384" extent="1-16" drill="0.35"/>
-<via x="13.2362" y="7.2136" extent="1-16" drill="0.35"/>
-<via x="13.4902" y="10.0076" extent="1-16" drill="0.35"/>
+<via x="13.1854" y="7.2136" extent="1-16" drill="0.35"/>
 <via x="8.6642" y="6.2992" extent="1-16" drill="0.35"/>
+<via x="3.381" y="11.4808" extent="1-16" drill="0.35"/>
+<via x="13.8204" y="8.8138" extent="1-16" drill="0.35"/>
+<via x="9.1976" y="9.4488" extent="1-16" drill="0.35"/>
+<via x="16.8176" y="6.4008" extent="1-16" drill="0.35"/>
+<via x="8.9436" y="23.6728" extent="1-16" drill="0.35"/>
+<via x="3.3556" y="8.4328" extent="1-16" drill="0.35"/>
 </signal>
 <signal name="+3V3">
@@
 <contactref element="U$3" pad="PA10"/>
 <contactref element="J1" pad="22"/>
-<wire x1="2.9416" y1="1.3716" x2="1.8418" y2="2.4714" width="0.254" layer="1"/>
-<wire x1="2.9416" y1="1.3716" x2="11.9634" y2="1.3716" width="0.254" layer="1"/>
-<wire x1="12.3952" y1="1.8034" x2="11.9634" y2="1.3716" width="0.254" layer="1"/>
-<wire x1="15.4302" y1="11.5406" x2="15.4302" y2="8.369" width="0.254" layer="1"/>
-<wire x1="15.4302" y1="8.369" x2="13.4366" y2="6.3754" width="0.254" layer="1"/>
-<wire x1="13.4366" y1="6.3754" x2="12.6492" y2="6.3754" width="0.254" layer="1"/>
-<wire x1="12.6492" y1="6.3754" x2="12.3952" y2="6.1214" width="0.254" layer="1"/>
-<wire x1="12.3952" y1="6.1214" x2="12.3952" y2="1.8034" width="0.254" layer="1"/>
+<wire x1="2.8908" y1="1.4224" x2="1.8418" y2="2.4714" width="0.254" layer="1"/>
+<wire x1="2.8908" y1="1.4224" x2="11.5824" y2="1.4224" width="0.254" layer="1"/>
+<wire x1="12.3444" y1="2.1844" x2="11.5824" y2="1.4224" width="0.254" layer="1"/>
+<wire x1="15.4302" y1="11.5406" x2="15.4302" y2="8.4706" width="0.254" layer="1"/>
+<wire x1="15.4302" y1="8.4706" x2="13.335" y2="6.3754" width="0.254" layer="1"/>
+<wire x1="13.335" y1="6.3754" x2="12.6492" y2="6.3754" width="0.254" layer="1"/>
+<wire x1="12.6492" y1="6.3754" x2="12.3444" y2="6.0706" width="0.254" layer="1"/>
+<wire x1="12.3444" y1="6.0706" x2="12.3444" y2="2.1844" width="0.254" layer="1"/>
 </signal>
 <signal name="CLK">
 <contactref element="U$3" pad="PA9"/>
 <contactref element="J1" pad="20"/>
-<wire x1="1.8418" y1="4.4714" x2="2.8314" y2="5.461" width="0.254" layer="1"/>
-<wire x1="9.1948" y1="5.461" x2="11.6332" y2="7.8994" width="0.254" layer="1"/>
-<wire x1="11.6332" y1="7.8994" x2="12.9032" y2="7.8994" width="0.254" layer="1"/>
-<wire x1="12.9032" y1="7.8994" x2="14.6302" y2="9.6264" width="0.254" layer="1"/>
-<wire x1="2.8314" y1="5.461" x2="9.1948" y2="5.461" width="0.254" layer="1"/>
-<wire x1="14.6302" y1="9.6264" x2="14.6302" y2="11.5406" width="0.254" layer="1"/>
+<wire x1="9.2964" y1="5.461" x2="3.0854" y2="5.461" width="0.254" layer="1"/>
+<wire x1="1.8418" y1="4.4714" x2="2.0958" y2="4.4714" width="0.254" layer="1"/>
+<wire x1="3.0854" y1="5.461" x2="2.0958" y2="4.4714" width="0.254" layer="1"/>
+<wire x1="14.6302" y1="11.5406" x2="14.6302" y2="10.7948" width="0.254" layer="1"/>
+<wire x1="14.3256" y1="10.4902" x2="12.3698" y2="10.4902" width="0.254" layer="1"/>
+<wire x1="12.3698" y1="10.4902" x2="12.0904" y2="10.2108" width="0.254" layer="1"/>
+<wire x1="12.0904" y1="9.7536" x2="12.319" y2="9.525" width="0.254" layer="1"/>
+<wire x1="12.319" y1="9.525" x2="14.478" y2="9.525" width="0.254" layer="1"/>
+<wire x1="14.6302" y1="10.7948" x2="14.3256" y2="10.4902" width="0.254" layer="1"/>
+<wire x1="12.0904" y1="10.2108" x2="12.0904" y2="9.7536" width="0.254" layer="1"/>
+<wire x1="14.478" y1="9.525" x2="14.840509375" y2="9.162490625" width="0.254" layer="1"/>
+<wire x1="14.840509375" y1="9.162490625" x2="14.840509375" y2="8.527490625" width="0.254" layer="1"/>
+<wire x1="14.39021875" y1="8.0772" x2="11.9126" y2="8.0772" width="0.254" layer="1"/>
+<wire x1="11.9126" y1="8.0772" x2="9.2964" y2="5.461" width="0.254" layer="1"/>
+<wire x1="14.840509375" y1="8.527490625" x2="14.39021875" y2="8.0772" width="0.254" layer="1"/>
 </signal>
 <signal name="GPIO7">
@@
 <contactref element="U$3" pad="PB4"/>
 <contactref element="J1" pad="18"/>
-<wire x1="20.0802" y1="14.5906" x2="18.9848" y2="14.5906" width="0.254" layer="1"/>
-<wire x1="18.9848" y1="14.5906" x2="18.9738" y2="14.5796" width="0.254" layer="1"/>
-<via x="18.9738" y="14.5796" extent="1-16" drill="0.35"/>
-<wire x1="18.9738" y1="14.5796" x2="17.018" y2="12.6238" width="0.254" layer="16"/>
-<wire x1="17.018" y1="12.6238" x2="10.5664" y2="12.6238" width="0.254" layer="16"/>
+<wire x1="20.0802" y1="14.5906" x2="19.0102" y2="14.5906" width="0.254" layer="1"/>
+<wire x1="19.0102" y1="14.5906" x2="17.2466" y2="12.827" width="0.254" layer="1"/>
+<via x="17.2466" y="12.827" extent="1-16" drill="0.35"/>
+<wire x1="17.2466" y1="12.827" x2="17.0434" y2="12.6238" width="0.254" layer="16"/>
+<wire x1="17.0434" y1="12.6238" x2="10.5664" y2="12.6238" width="0.254" layer="16"/>
 <wire x1="10.5664" y1="12.6238" x2="5.4102" y2="7.4676" width="0.254" layer="16"/>
 <wire x1="5.4102" y1="7.4676" x2="2.838" y2="7.4676" width="0.254" layer="16"/>
@@
 <contactref element="J1" pad="17"/>
 <wire x1="4.8638" y1="6.4714" x2="5.0744" y2="6.4714" width="0.254" layer="16"/>
-<wire x1="17.526" y1="12.1412" x2="18.9738" y2="13.589" width="0.254" layer="16"/>
-<via x="18.9738" y="13.589" extent="1-16" drill="0.35"/>
-<wire x1="19.1754" y1="13.7906" x2="18.9738" y2="13.589" width="0.254" layer="1"/>
-<wire x1="19.1754" y1="13.7906" x2="20.0802" y2="13.7906" width="0.254" layer="1"/>
+<wire x1="17.6022" y1="12.1412" x2="18.161" y2="12.7" width="0.254" layer="16"/>
+<via x="18.161" y="12.7" extent="1-16" drill="0.35"/>
+<wire x1="19.2516" y1="13.7906" x2="18.161" y2="12.7" width="0.254" layer="1"/>
+<wire x1="19.2516" y1="13.7906" x2="20.0802" y2="13.7906" width="0.254" layer="1"/>
 <wire x1="5.0744" y1="6.4714" x2="10.7442" y2="12.1412" width="0.254" layer="16"/>
-<wire x1="10.7442" y1="12.1412" x2="17.526" y2="12.1412" width="0.254" layer="16"/>
+<wire x1="10.7442" y1="12.1412" x2="17.6022" y2="12.1412" width="0.254" layer="16"/>
 </signal>
 <signal name="NRST">
@@
 <wire x1="10.1854" y1="12.2428" x2="10.1854" y2="14.0716" width="0.254" layer="1"/>
 </signal>
+<signal name="NO">
+<polygon width="0.0254" layer="16" pour="cutout">
+<vertex x="12.4714" y="13.716"/>
+<vertex x="12.4714" y="12.954"/>
+<vertex x="12.446" y="12.954"/>
+<vertex x="12.446" y="13.716"/>
+</polygon>
+</signal>
 </signals>

Commit message: Pretty much ready for production (owo)
Parts:
- moved C4 9.37 mm to (16.4, 16.7), turned to 180 degrees
- moved C2 7.06 mm to (16.4, 15.2), turned to 180 degrees
- moved C5 6.45 mm to (16.4, 23.0)
- moved C6 6.40 mm to (16.4, 24.4)
- moved C3 4.85 mm to (16.3, 20.2), turned to 90 degrees
- moved C1 2.95 mm to (17.8, 20.2), turned to 90 degrees
- moved R1 1.43 mm to (9.25, 23.4), turned to 180 degrees
- moved U$3 1.02 mm to (12.0, 20.0)
- moved C11 0.84 mm to (11.2, 4.34)
- moved R3 0.42 mm to (16.4, 23.0)
- moved R4 0.06 mm to (8.69, 7.67)
Connections:
- net +3V3: now also J1.4; no longer J1.6
- net GND: now also J1.6; no longer J1.4
Routing:
- net +3V3: track 72.2 -> 68.1 mm, vias 4 -> 6
- net GND: track 7.00 -> 3.89 mm, vias 28 -> 27
- net N$2: track 7.17 -> 5.64 mm
- net GPIO5: track 4.38 -> 2.97 mm
- net GPIO3: track 4.68 -> 3.36 mm
- net GPIO6: track 4.42 -> 3.10 mm
- net GPIO1: track 5.33 -> 4.20 mm
- net ALERT2: track 18.2 -> 17.2 mm
- net LED: track 5.62 -> 6.64 mm
- net ALERT1: track 21.6 -> 20.6 mm
- net SWDIO: track 5.01 -> 6.03 mm
- net NRST: track 19.6 -> 20.6 mm
- net CLK: track 22.3 -> 21.5 mm
- net GPIO4: track 4.48 -> 3.73 mm
- net CAN_TX: track 11.6 -> 11.1 mm
- added copper zone on layer 1, net NO

Commit message: OWO
Parts:
- moved R4 2.29 mm to (7.49, 9.63), turned to 225 degrees
- moved R5 0.75 mm to (7.29, 11.5), turned to 225 degrees
Routing:
- net N$1: track 7.99 -> 5.60 mm
- net N$2: track 5.64 -> 4.43 mm
- net C2_2: track 3.30 -> 2.26 mm
- net GPIO4: track 3.73 -> 3.16 mm
